Commit message: 03/06/2026

File: robot_urdf/urdf/robot.SLDASM.urdf (robot description, URDF)
Before this commit: robot robot.SLDASM, 15 links, 16 joints
Links:
- link base_link: geometry visual mesh filename=../meshes/base_link.STL
- link calf_left_link_1: geometry visual mesh filename=../meshes/calf_left_link_1.STL
- link calf_left_link_2: geometry visual mesh filename=../meshes/calf_left_link_2.STL
- link calf_right_link_1: geometry visual mesh filename=../meshes/calf_right_link_1.STL
- link calf_right_link_2: geometry visual mesh filename=../meshes/calf_right_link_2.STL
- link hip_frame_link_left: geometry visual mesh filename=../meshes/hip_frame_link_left.STL
- link hip_frame_link_right: geometry visual mesh filename=../meshes/hip_frame_link_right.STL
- link pad_link_left: geometry visual mesh filename=../meshes/pad_link_left.STL
- link pad_link_right: geometry visual mesh filename=../meshes/pad_link_right.STL
- link thigh_left_1: geometry visual mesh filename=../meshes/thigh_left_1.STL
- link thigh_left_2: geometry visual mesh filename=../meshes/thigh_left_2.STL
- link thigh_right_1: geometry visual mesh filename=../meshes/thigh_right_1.STL
- link thigh_right_2: geometry visual mesh filename=../meshes/thigh_right_2.STL
- link wheel_link_left: geometry visual mesh filename=../meshes/wheel_link_left.STL
- link wheel_link_right: geometry visual mesh filename=../meshes/wheel_link_right.STL
